Commit message: Add teleop

File: src/amr_description/urdf/amr.urdf.xacro (robot description, xacro)
@@ -7,30 +7,31 @@
   <xacro:property name="wheel_radius" value="0.05"/>
   <xacro:property name="wheel_width"  value="0.03"/>
-  <xacro:property name="wheel_sep"    value="0.24"/> <!-- center-to-center -->
+  <xacro:property name="wheel_y" value="${base_width/2 + wheel_width/2}"/>
+  <xacro:property name="wheel_sep" value="${2*wheel_y}"/>
   <!-- Materials -->
   <material name="gray"><color rgba="0.6 0.6 0.6 1.0"/></material>
   <material name="black"><color rgba="0.1 0.1 0.1 1.0"/></material>
   <!-- Base link -->
-<link name="base_link">
-  <visual>
-    <origin xyz="0 0 ${base_height/2 + wheel_radius}" rpy="0 0 0"/>
-    <geometry>
-      <box size="${base_length} ${base_width} ${base_height}"/>
-    </geometry>
-    <material name="gray"/>
-  </visual>
-  <collision>
-    <origin xyz="0 0 ${base_height/2 + wheel_radius}" rpy="0 0 0"/>
-    <geometry>
-      <box size="${base_length} ${base_width} ${base_height}"/>
-    </geometry>
-  </collision>
-  <inertial>
-    <origin xyz="0 0 ${base_height/2 + wheel_radius}" rpy="0 0 0"/>
-    <mass value="8.0"/>
-    <inertia ixx="0.12" ixy="0.0" ixz="0.0" iyy="0.20" iyz="0.0" izz="0.25"/>
-  </inertial>
-</link>
-  <!-- Wheels -->
+  <link name="base_link">
+    <visual>
+      <origin xyz="0 0 ${base_height/2 + wheel_radius}" rpy="0 0 0"/>
+      <geometry>
+        <box size="${base_length} ${base_width} ${base_height}"/>
+      </geometry>
+      <material name="gray"/>
+    </visual>
+    <collision>
+      <origin xyz="0 0 ${base_height/2 + wheel_radius}" rpy="0 0 0"/>
+      <geometry>
+        <box size="${base_length} ${base_width} ${base_height}"/>
+      </geometry>
+    </collision>
+    <inertial>
+      <origin xyz="0 0 ${base_height/2 + wheel_radius}" rpy="0 0 0"/>
+      <mass value="8.0"/>
+      <inertia ixx="0.12" ixy="0.0" ixz="0.0" iyy="0.20" iyz="0.0" izz="0.25"/>
+    </inertial>
+  </link>
+  <!-- Wheels (UPDATED: add collision + inertial) -->
   <link name="left_wheel_link">
     <visual>
@@ -41,4 +42,16 @@
       <material name="black"/>
     </visual>
+    <collision>
+      <origin xyz="0 0 0" rpy="1.5708 0 0"/>
+      <geometry>
+        <cylinder radius="${wheel_radius}" length="${wheel_width}"/>
+      </geometry>
+    </collision>
+    <inertial>
+      <origin xyz="0 0 0" rpy="0 0 0"/>
+      <mass value="0.5"/>
+      <!-- placeholder inertia; good enough for M2 -->
+      <inertia ixx="0.001" ixy="0.0" ixz="0.0" iyy="0.001" iyz="0.0" izz="0.001"/>
+    </inertial>
   </link>
   <link name="right_wheel_link">
@@ -50,4 +63,15 @@
       <material name="black"/>
     </visual>
+    <collision>
+      <origin xyz="0 0 0" rpy="1.5708 0 0"/>
+      <geometry>
+        <cylinder radius="${wheel_radius}" length="${wheel_width}"/>
+      </geometry>
+    </collision>
+    <inertial>
+      <origin xyz="0 0 0" rpy="0 0 0"/>
+      <mass value="0.5"/>
+      <inertia ixx="0.001" ixy="0.0" ixz="0.0" iyy="0.001" iyz="0.0" izz="0.001"/>
+    </inertial>
   </link>
   <!-- Wheel joints -->
@@ -55,5 +79,5 @@
     <parent link="base_link"/>
     <child link="left_wheel_link"/>
-    <origin xyz="0 ${wheel_sep/2} ${wheel_radius}" rpy="0 0 0"/>
+    <origin xyz="0 ${wheel_y} ${wheel_radius}" rpy="0 0 0"/>
     <axis xyz="0 1 0"/>
   </joint>
@@ -61,9 +85,15 @@
     <parent link="base_link"/>
     <child link="right_wheel_link"/>
-    <origin xyz="0 -${wheel_sep/2} ${wheel_radius}" rpy="0 0 0"/>
+    <origin xyz="0 -${wheel_y} ${wheel_radius}" rpy="0 0 0"/>
     <axis xyz="0 1 0"/>
   </joint>
-  <!-- A forward-facing lidar frame placeholder (sensor added later) -->
-  <link name="lidar_link"/>
+  <!-- Lidar frame placeholder (UPDATED: give inertial so Gazebo doesn't complain) -->
+  <link name="lidar_link">
+    <inertial>
+      <origin xyz="0 0 0" rpy="0 0 0"/>
+      <mass value="0.1"/>
+      <inertia ixx="1e-5" ixy="0.0" ixz="0.0" iyy="1e-5" iyz="0.0" izz="1e-5"/>
+    </inertial>
+  </link>
   <joint name="lidar_joint" type="fixed">
     <parent link="base_link"/>
@@ -71,3 +101,38 @@
     <origin xyz="${base_length/2 - 0.05} 0 ${base_height + 0.02}" rpy="0 0 0"/>
   </joint>
+  <!-- ros2_control -->
+  <ros2_control name="MockSystem" type="system">
+    <hardware>
+      <plugin>mock_components/GenericSystem</plugin>
+    </hardware>
+    <joint name="left_wheel_joint">
+      <command_interface name="velocity"/>
+      <state_interface name="position"/>
+      <state_interface name="velocity"/>
+    </joint>
+    <joint name="right_wheel_joint">
+      <command_interface name="velocity"/>
+      <state_interface name="position"/>
+      <state_interface name="velocity"/>
+    </joint>
+  </ros2_control>
+  <!-- Gazebo plugin hook -->
+  <gazebo>
+    <!-- <plugin name="gazebo_ros2_control" filename="libgazebo_ros2_control.so"> -->
+      <!-- Where Gazebo should read the robot_description from -->
+      <robot_param>robot_description</robot_param>
+      <robot_param_node>/robot_state_publisher</robot_param_node>
+      <!-- Load controller params directly into the Gazebo controller manager -->
+      <parameters>$(find amr_control)/config/diff_drive_controller.yaml</parameters>
+    </plugin>
+  </gazebo>
+  <!-- OPTIONAL but recommended: wheel friction (reduces sliding in M2) -->
+  <gazebo reference="left_wheel_link">
+    <mu1>1.0</mu1>
+    <mu2>1.0</mu2>
+  </gazebo>
+  <gazebo reference="right_wheel_link">
+    <mu1>1.0</mu1>
+    <mu2>1.0</mu2>
+  </gazebo>
 </robot>

Commit message: Fix URDF bugs

File: src/amr_description/urdf/amr.urdf.xacro (robot description, xacro)
@@ -1,5 +1,4 @@
 <?xml version="1.0"?>
 <robot xmlns:xacro="http://www.ros.org/wiki/xacro" name="amr">
-  <!-- Parameters -->
   <xacro:property name="base_length" value="0.35"/>
   <xacro:property name="base_width"  value="0.28"/>
@@ -9,8 +8,12 @@
   <xacro:property name="wheel_y" value="${base_width/2 + wheel_width/2}"/>
   <xacro:property name="wheel_sep" value="${2*wheel_y}"/>
-  <!-- Materials -->
   <material name="gray"><color rgba="0.6 0.6 0.6 1.0"/></material>
   <material name="black"><color rgba="0.1 0.1 0.1 1.0"/></material>
-  <!-- Base link -->
+  <link name="base_footprint"/>
+  <joint name="base_joint" type="fixed">
+    <parent link="base_footprint"/>
+    <child link="base_link"/>
+    <origin xyz="0 0 0" rpy="0 0 0"/>
+  </joint>
   <link name="base_link">
     <visual>
@@ -33,5 +36,4 @@
     </inertial>
   </link>
-  <!-- Wheels (UPDATED: add collision + inertial) -->
   <link name="left_wheel_link">
     <visual>
@@ -51,8 +53,13 @@
       <origin xyz="0 0 0" rpy="0 0 0"/>
       <mass value="0.5"/>
-      <!-- placeholder inertia; good enough for M2 -->
       <inertia ixx="0.001" ixy="0.0" ixz="0.0" iyy="0.001" iyz="0.0" izz="0.001"/>
     </inertial>
   </link>
+  <joint name="left_wheel_joint" type="continuous">
+    <parent link="base_link"/>
+    <child link="left_wheel_link"/>
+    <origin xyz="0 ${wheel_y} ${wheel_radius}" rpy="0 0 0"/>
+    <axis xyz="0 1 0"/>
+  </joint>
   <link name="right_wheel_link">
     <visual>
@@ -75,11 +82,4 @@
     </inertial>
   </link>
-  <!-- Wheel joints -->
-  <joint name="left_wheel_joint" type="continuous">
-    <parent link="base_link"/>
-    <child link="left_wheel_link"/>
-    <origin xyz="0 ${wheel_y} ${wheel_radius}" rpy="0 0 0"/>
-    <axis xyz="0 1 0"/>
-  </joint>
   <joint name="right_wheel_joint" type="continuous">
     <parent link="base_link"/>
@@ -88,5 +88,22 @@
     <axis xyz="0 1 0"/>
   </joint>
-  <!-- Lidar frame placeholder (UPDATED: give inertial so Gazebo doesn't complain) -->
+  <link name="front_caster">
+    <visual>
+      <geometry><sphere radius="0.05"/></geometry>
+      <material name="black"/>
+    </visual>
+    <collision>
+      <geometry><sphere radius="0.05"/></geometry>
+    </collision>
+    <inertial>
+      <mass value="0.1"/>
+      <inertia ixx="0.0001" ixy="0.0" ixz="0.0" iyy="0.0001" iyz="0.0" izz="0.0001"/>
+    </inertial>
+  </link>
+  <joint name="front_caster_joint" type="fixed">
+    <parent link="base_link"/>
+    <child link="front_caster"/>
+    <origin xyz="0.12 0 0.05" rpy="0 0 0"/>
+  </joint>
   <link name="lidar_link">
     <inertial>
@@ -101,8 +118,7 @@
     <origin xyz="${base_length/2 - 0.05} 0 ${base_height + 0.02}" rpy="0 0 0"/>
   </joint>
-  <!-- ros2_control -->
-  <ros2_control name="MockSystem" type="system">
+  <ros2_control name="GazeboSystem" type="system">
     <hardware>
-      <plugin>mock_components/GenericSystem</plugin>
+      <plugin>gazebo_ros2_control/GazeboSystem</plugin>
     </hardware>
     <joint name="left_wheel_joint">
@@ -117,15 +133,12 @@
     </joint>
   </ros2_control>
-  <!-- Gazebo plugin hook -->
   <gazebo>
-    <!-- <plugin name="gazebo_ros2_control" filename="libgazebo_ros2_control.so"> -->
-      <!-- Where Gazebo should read the robot_description from -->
-      <robot_param>robot_description</robot_param>
-      <robot_param_node>/robot_state_publisher</robot_param_node>
-      <!-- Load controller params directly into the Gazebo controller manager -->
+    <plugin name="gazebo_ros2_control" filename="libgazebo_ros2_control.so">
       <parameters>$(find amr_control)/config/diff_drive_controller.yaml</parameters>
+      <ros>
+        <namespace>/</namespace>
+      </ros>
     </plugin>
   </gazebo>
-  <!-- OPTIONAL but recommended: wheel friction (reduces sliding in M2) -->
   <gazebo reference="left_wheel_link">
     <mu1>1.0</mu1>
@@ -136,3 +149,7 @@
     <mu2>1.0</mu2>
   </gazebo>
+  <gazebo reference="front_caster">
+    <mu1>0.001</mu1>
+    <mu2>0.001</mu2>
+  </gazebo>
 </robot>
